File: controllerpro.sch (EAGLE design)
At the start: 10 parts, among them IC1 MCP1703CB, IC2 741G3157DBVR, IC3 741G3157DBVR, IC4 741G3157DBVR, IC5 741G3157DBVR

Commit message: Now smaller!  Rearranged things to minimize size
Mostly to reduce board cost, but hey!
Parts:
- removed _1: TEENSY, teensy:TEENSY
- added U$5: TEENSY_HEADERS, teensy:TEENSY_HEADERS
Connections:
- net N$11 renamed V33
- net DATA0: now also U$5._D3; no longer _1._D0
- net DATA1: now also U$5._D2; no longer _1._D1
- net DATA2: now also U$5._D1; no longer _1._D2
- net DATA3: now also U$5._D0; no longer _1._D3
- net N$1: now also U$5._D7; no longer _1._D7
- net N$2: now also U$5._D6; no longer _1._D6
- net N64_OR_NES0: now also U$5._B3; no longer _1._B0
- net N64_OR_NES1: now also U$5._B2; no longer _1._B1
- net N64_OR_NES2: now also U$5._B1; no longer _1._B2
- net N64_OR_NES3: now also U$5._B0; no longer _1._B3
- net S_OR_NES0: now also U$5._F7; no longer _1._F4
- net S_OR_NES1: now also U$5._F6; no longer _1._F5
- net S_OR_NES2: now also U$5._F5; no longer _1._F6
- net S_OR_NES3: now also U$5._F4; no longer _1._F7
- net VCC: now also U$5.5V; no longer _1.5V
Changed lines of the file:
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@@
 <class number="0" name="default" width="0" drill="0">
+</class>
+<class number="1" name="VCC" width="0.3048" drill="0">
+</class>
+<class number="2" name="GND" width="0.3048" drill="0">
 </class>
 </classes>
 <parts>
-<part name="_1" library="teensy" deviceset="TEENSY" device=""/>
 <part name="U$1" library="custom" deviceset="NINTENDO-MULTI" device=""/>
 <part name="U$2" library="custom" deviceset="NINTENDO-MULTI" device=""/>
@@
 <part name="SUPPLY4" library="supply2" deviceset="VCC" device=""/>
 <part name="SUPPLY5" library="supply2" deviceset="GND" device=""/>
+<part name="U$5" library="teensy" deviceset="TEENSY_HEADERS" device=""/>
 </parts>
 <sheets>
@@
 </plain>
 <instances>
-<instance part="_1" gate="G$1" x="53.34" y="53.34" rot="R180"/>
 <instance part="U$1" gate="G$1" x="121.92" y="86.36" rot="R270"/>
 <instance part="U$2" gate="G$1" x="116.84" y="55.88" rot="R270"/>
@@
 <instance part="SUPPLY4" gate="G$1" x="-25.4" y="121.92"/>
 <instance part="SUPPLY5" gate="GND" x="-25.4" y="96.52"/>
+<instance part="U$5" gate="G$1" x="53.34" y="53.34" rot="R180"/>
 </instances>
 <busses>
@@
 <net name="N$1" class="0">
 <segment>
-<pinref part="_1" gate="G$1" pin="_D7"/>
 <wire x1="66.04" y1="43.18" x2="78.74" y2="43.18" width="0.1524" layer="91"/>
 <wire x1="78.74" y1="43.18" x2="78.74" y2="63.5" width="0.1524" layer="91"/>
@@
 <wire x1="154.94" y1="73.66" x2="78.74" y2="73.66" width="0.1524" layer="91"/>
 <junction x="78.74" y="73.66"/>
+<pinref part="U$5" gate="G$1" pin="_D7"/>
 </segment>
 </net>
 <net name="N$2" class="0">
 <segment>
-<pinref part="_1" gate="G$1" pin="_D6"/>
 <wire x1="66.04" y1="40.64" x2="81.28" y2="40.64" width="0.1524" layer="91"/>
 <wire x1="81.28" y1="91.44" x2="81.28" y2="71.12" width="0.1524" layer="91"/>
@@
 <pinref part="U$3" gate="G$1" pin="3"/>
 <wire x1="81.28" y1="71.12" x2="154.94" y2="71.12" width="0.1524" layer="91"/>
+<pinref part="U$5" gate="G$1" pin="_D6"/>
 </segment>
 </net>
@@
 <segment>
 <pinref part="SUPPLY2" gate="G$1" pin="VCC"/>
-<pinref part="_1" gate="G$1" pin="5V"/>
 <wire x1="35.56" y1="20.32" x2="40.64" y2="20.32" width="0.1524" layer="91"/>
+<pinref part="U$5" gate="G$1" pin="5V"/>
 </segment>
 <segment>
@@
 </segment>
 </net>
-<net name="N$11" class="0">
+<net name="V33" class="0">
 <segment>
 <wire x1="170.18" y1="114.3" x2="127" y2="114.3" width="0.1524" layer="91"/>
@@
 <net name="N64_OR_NES0" class="0">
 <segment>
-<pinref part="_1" gate="G$1" pin="_B0"/>
-<wire x1="40.64" y1="38.1" x2="30.48" y2="38.1" width="0.1524" layer="91"/>
-</segment>
-<segment>
 <pinref part="IC2" gate="G$1" pin="!A!/B"/>
 <wire x1="109.22" y1="111.76" x2="109.22" y2="88.9" width="0.1524" layer="91"/>
 </segment>
+<segment>
+<pinref part="U$5" gate="G$1" pin="_B3"/>
+<wire x1="40.64" y1="30.48" x2="30.48" y2="30.48" width="0.1524" layer="91"/>
+</segment>
 </net>
 <net name="N64_OR_NES1" class="0">
-<segment>
-<pinref part="_1" gate="G$1" pin="_B1"/>
-<wire x1="40.64" y1="35.56" x2="30.48" y2="35.56" width="0.1524" layer="91"/>
-</segment>
 <segment>
 <wire x1="86.36" y1="111.76" x2="86.36" y2="66.04" width="0.1524" layer="91"/>
@@
 <wire x1="109.22" y1="66.04" x2="109.22" y2="58.42" width="0.1524" layer="91"/>
 </segment>
+<segment>
+<pinref part="U$5" gate="G$1" pin="_B2"/>
+<wire x1="40.64" y1="33.02" x2="30.48" y2="33.02" width="0.1524" layer="91"/>
+</segment>
 </net>
 <net name="N64_OR_NES2" class="0">
-<segment>
-<pinref part="_1" gate="G$1" pin="_B2"/>
-<wire x1="40.64" y1="33.02" x2="30.48" y2="33.02" width="0.1524" layer="91"/>
-</segment>
 <segment>
 <pinref part="IC4" gate="G$1" pin="!A!/B"/>
 <wire x1="147.32" y1="68.58" x2="147.32" y2="111.76" width="0.1524" layer="91"/>
 </segment>
+<segment>
+<pinref part="U$5" gate="G$1" pin="_B1"/>
+<wire x1="40.64" y1="35.56" x2="30.48" y2="35.56" width="0.1524" layer="91"/>
+</segment>
 </net>
 <net name="N64_OR_NES3" class="0">
-<segment>
-<pinref part="_1" gate="G$1" pin="_B3"/>
-<wire x1="40.64" y1="30.48" x2="30.48" y2="30.48" width="0.1524" layer="91"/>
-</segment>
 <segment>
 <pinref part="IC5" gate="G$1" pin="!A!/B"/>
 <wire x1="152.4" y1="38.1" x2="152.4" y2="111.76" width="0.1524" layer="91"/>
 </segment>
+<segment>
+<pinref part="U$5" gate="G$1" pin="_B0"/>
+<wire x1="40.64" y1="38.1" x2="30.48" y2="38.1" width="0.1524" layer="91"/>
+</segment>
 </net>
 <net name="S_OR_NES0" class="0">
-<segment>
-<pinref part="_1" gate="G$1" pin="_F4"/>
-<wire x1="40.64" y1="63.5" x2="33.02" y2="63.5" width="0.1524" layer="91"/>
-</segment>
 <segment>
 <pinref part="U$1" gate="G$1" pin="1"/>
 <wire x1="119.38" y1="96.52" x2="119.38" y2="109.22" width="0.1524" layer="91"/>
 </segment>
+<segment>
+<pinref part="U$5" gate="G$1" pin="_F7"/>
+<wire x1="40.64" y1="71.12" x2="33.02" y2="71.12" width="0.1524" layer="91"/>
+</segment>
 </net>
 <net name="S_OR_NES1" class="0">
-<segment>
-<pinref part="_1" gate="G$1" pin="_F5"/>
-<wire x1="40.64" y1="66.04" x2="33.02" y2="66.04" width="0.1524" layer="91"/>
-</segment>
 <segment>
 <pinref part="U$2" gate="G$1" pin="1"/>
 <wire x1="114.3" y1="66.04" x2="114.3" y2="109.22" width="0.1524" layer="91"/>
 </segment>
+<segment>
+<pinref part="U$5" gate="G$1" pin="_F6"/>
+<wire x1="40.64" y1="68.58" x2="33.02" y2="68.58" width="0.1524" layer="91"/>
+</segment>
 </net>
 <net name="S_OR_NES2" class="0">
-<segment>
-<pinref part="_1" gate="G$1" pin="_F6"/>
-<wire x1="40.64" y1="68.58" x2="33.02" y2="68.58" width="0.1524" layer="91"/>
-</segment>
 <segment>
 <pinref part="U$3" gate="G$1" pin="1"/>
 <wire x1="154.94" y1="76.2" x2="154.94" y2="109.22" width="0.1524" layer="91"/>
 </segment>
+<segment>
+<pinref part="U$5" gate="G$1" pin="_F5"/>
+<wire x1="40.64" y1="66.04" x2="33.02" y2="66.04" width="0.1524" layer="91"/>
+</segment>
 </net>
 <net name="S_OR_NES3" class="0">
-<segment>
-<pinref part="_1" gate="G$1" pin="_F7"/>
-<wire x1="40.64" y1="71.12" x2="33.02" y2="71.12" width="0.1524" layer="91"/>
-</segment>
 <segment>
 <wire x1="162.56" y1="109.22" x2="162.56" y2="45.72" width="0.1524" layer="91"/>
 <pinref part="U$4" gate="G$1" pin="1"/>
 <wire x1="162.56" y1="45.72" x2="157.48" y2="45.72" width="0.1524" layer="91"/>
+</segment>
+<segment>
+<pinref part="U$5" gate="G$1" pin="_F4"/>
+<wire x1="40.64" y1="63.5" x2="33.02" y2="63.5" width="0.1524" layer="91"/>
 </segment>
 </net>
@@
 </segment>
 <segment>
-<pinref part="_1" gate="G$1" pin="_D0"/>
-<wire x1="66.04" y1="25.4" x2="71.12" y2="25.4" width="0.1524" layer="91"/>
+<pinref part="U$5" gate="G$1" pin="_D3"/>
+<wire x1="66.04" y1="33.02" x2="71.12" y2="33.02" width="0.1524" layer="91"/>
 </segment>
 </net>
@@
 </segment>
 <segment>
-<pinref part="_1" gate="G$1" pin="_D1"/>
-<wire x1="66.04" y1="27.94" x2="71.12" y2="27.94" width="0.1524" layer="91"/>
+<pinref part="U$5" gate="G$1" pin="_D2"/>
+<wire x1="66.04" y1="30.48" x2="71.12" y2="30.48" width="0.1524" layer="91"/>
 </segment>
 </net>
@@
 </segment>
 <segment>
-<pinref part="_1" gate="G$1" pin="_D2"/>
-<wire x1="66.04" y1="30.48" x2="71.12" y2="30.48" width="0.1524" layer="91"/>
+<pinref part="U$5" gate="G$1" pin="_D1"/>
+<wire x1="66.04" y1="27.94" x2="71.12" y2="27.94" width="0.1524" layer="91"/>
 </segment>
 </net>
@@
 </segment>
 <segment>
-<pinref part="_1" gate="G$1" pin="_D3"/>
-<wire x1="66.04" y1="33.02" x2="71.12" y2="33.02" width="0.1524" layer="91"/>
-</segment>
-</net>
+<pinref part="U$5" gate="G$1" pin="_D0"/>
+<wire x1="66.04" y1="25.4" x2="71.12" y2="25.4" width="0.1524" layer="91"/>
+</segment>
+</net>

Commit message: Add my custom teensy parts to the custom library
Just removed the unneeded pins, we'll just be using two headers
Parts:
- U$5: device teensy:TEENSY_HEADERS -> custom:TEENSY_HEADERS
Changed lines of the file:
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@@
 <part name="SUPPLY4" library="supply2" deviceset="VCC" device=""/>
 <part name="SUPPLY5" library="supply2" deviceset="GND" device=""/>
-<part name="U$5" library="teensy" deviceset="TEENSY_HEADERS" device=""/>
+<part name="U$5" library="custom" deviceset="TEENSY_HEADERS" device=""/>
 </parts>
 <sheets>

Commit message: Adding some net names, connecting a missing GND
Connections:
- net N$1 renamed CLOCK
- net N$2 renamed LATCH
- net GND: now also U$5._GND
Changed lines of the file:
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@@
 <part name="SUPPLY5" library="supply2" deviceset="GND" device=""/>
 <part name="U$5" library="custom" deviceset="TEENSY_HEADERS" device=""/>
+<part name="SUPPLY6" library="supply2" deviceset="GND" device=""/>
 </parts>
 <sheets>
@@
 <instance part="SUPPLY5" gate="GND" x="-25.4" y="96.52"/>
 <instance part="U$5" gate="G$1" x="53.34" y="53.34" rot="R180"/>
+<instance part="SUPPLY6" gate="GND" x="66.04" y="15.24"/>
 </instances>
 <busses>
@@
 </busses>
 <nets>
-<net name="N$1" class="0">
+<net name="CLOCK" class="0">
 <segment>
 <wire x1="66.04" y1="43.18" x2="78.74" y2="43.18" width="0.1524" layer="91"/>
@@
 </segment>
 </net>
-<net name="N$2" class="0">
+<net name="LATCH" class="0">
 <segment>
 <wire x1="66.04" y1="40.64" x2="81.28" y2="40.64" width="0.1524" layer="91"/>
@@
 <junction x="-25.4" y="101.6"/>
 </segment>
+<segment>
+<pinref part="SUPPLY6" gate="GND" pin="GND"/>
+<pinref part="U$5" gate="G$1" pin="_GND"/>
+<wire x1="66.04" y1="17.78" x2="66.04" y2="20.32" width="0.1524" layer="91"/>
+</segment>
 </net>

Commit message: Using only needed pins, also starting on wires
Parts:
- U$5: value TEENSY_HEADERS -> TEENSY_MC_PINS; device custom:TEENSY_HEADERS -> custom:TEENSY_MC_PINS
Changed lines of the file:
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@@
 <part name="SUPPLY4" library="supply2" deviceset="VCC" device=""/>
 <part name="SUPPLY5" library="supply2" deviceset="GND" device=""/>
-<part name="U$5" library="custom" deviceset="TEENSY_HEADERS" device=""/>
+<part name="U$5" library="custom" deviceset="TEENSY_MC_PINS" device=""/>
 <part name="SUPPLY6" library="supply2" deviceset="GND" device=""/>
 </parts>

Commit message: All wired up (intially)!
Connections:
- net DATA0: now also U$5._D2; no longer U$5._D3
- net DATA1: now also U$5._D3; no longer U$5._D2
- net DATA2: now also U$5._D0; no longer U$5._D1
- net DATA3: now also U$5._D1; no longer U$5._D0
- net N64_OR_NES0: now also U$5._B2; no longer U$5._B3
- net N64_OR_NES1: now also U$5._B3; no longer U$5._B2
- net N64_OR_NES2: now also U$5._B0; no longer U$5._B1
- net N64_OR_NES3: now also U$5._B1; no longer U$5._B0
- net S_OR_NES0: now also U$5._F6; no longer U$5._F7
- net S_OR_NES1: now also U$5._F7; no longer U$5._F6
- net S_OR_NES2: now also U$5._F4; no longer U$5._F5
- net S_OR_NES3: now also U$5._F5; no longer U$5._F4
Changed lines of the file:
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@@
 </segment>
 <segment>
-<pinref part="U$5" gate="G$1" pin="_B3"/>
-<wire x1="40.64" y1="30.48" x2="30.48" y2="30.48" width="0.1524" layer="91"/>
+<pinref part="U$5" gate="G$1" pin="_B2"/>
+<wire x1="40.64" y1="33.02" x2="30.48" y2="33.02" width="0.1524" layer="91"/>
 </segment>
 </net>
@@
 </segment>
 <segment>
-<pinref part="U$5" gate="G$1" pin="_B2"/>
-<wire x1="40.64" y1="33.02" x2="30.48" y2="33.02" width="0.1524" layer="91"/>
+<pinref part="U$5" gate="G$1" pin="_B3"/>
+<wire x1="40.64" y1="30.48" x2="30.48" y2="30.48" width="0.1524" layer="91"/>
 </segment>
 </net>
@@
 </segment>
 <segment>
-<pinref part="U$5" gate="G$1" pin="_B1"/>
-<wire x1="40.64" y1="35.56" x2="30.48" y2="35.56" width="0.1524" layer="91"/>
+<pinref part="U$5" gate="G$1" pin="_B0"/>
+<wire x1="40.64" y1="38.1" x2="30.48" y2="38.1" width="0.1524" layer="91"/>
 </segment>
 </net>
@@
 </segment>
 <segment>
-<pinref part="U$5" gate="G$1" pin="_B0"/>
-<wire x1="40.64" y1="38.1" x2="30.48" y2="38.1" width="0.1524" layer="91"/>
+<pinref part="U$5" gate="G$1" pin="_B1"/>
+<wire x1="40.64" y1="35.56" x2="30.48" y2="35.56" width="0.1524" layer="91"/>
 </segment>
 </net>
@@
 </segment>
 <segment>
-<pinref part="U$5" gate="G$1" pin="_F7"/>
-<wire x1="40.64" y1="71.12" x2="33.02" y2="71.12" width="0.1524" layer="91"/>
+<pinref part="U$5" gate="G$1" pin="_F6"/>
+<wire x1="40.64" y1="68.58" x2="33.02" y2="68.58" width="0.1524" layer="91"/>
 </segment>
 </net>
@@
 </segment>
 <segment>
-<pinref part="U$5" gate="G$1" pin="_F6"/>
-<wire x1="40.64" y1="68.58" x2="33.02" y2="68.58" width="0.1524" layer="91"/>
+<pinref part="U$5" gate="G$1" pin="_F7"/>
+<wire x1="40.64" y1="71.12" x2="33.02" y2="71.12" width="0.1524" layer="91"/>
 </segment>
 </net>
@@
 </segment>
 <segment>
-<pinref part="U$5" gate="G$1" pin="_F5"/>
-<wire x1="40.64" y1="66.04" x2="33.02" y2="66.04" width="0.1524" layer="91"/>
+<pinref part="U$5" gate="G$1" pin="_F4"/>
+<wire x1="40.64" y1="63.5" x2="33.02" y2="63.5" width="0.1524" layer="91"/>
 </segment>
 </net>
@@
 </segment>
 <segment>
-<pinref part="U$5" gate="G$1" pin="_F4"/>
-<wire x1="40.64" y1="63.5" x2="33.02" y2="63.5" width="0.1524" layer="91"/>
+<pinref part="U$5" gate="G$1" pin="_F5"/>
+<wire x1="40.64" y1="66.04" x2="33.02" y2="66.04" width="0.1524" layer="91"/>
 </segment>
 </net>
@@
 </segment>
 <segment>
-<pinref part="U$5" gate="G$1" pin="_D3"/>
-<wire x1="66.04" y1="33.02" x2="71.12" y2="33.02" width="0.1524" layer="91"/>
+<pinref part="U$5" gate="G$1" pin="_D2"/>
+<wire x1="66.04" y1="30.48" x2="71.12" y2="30.48" width="0.1524" layer="91"/>
 </segment>
 </net>
@@
 </segment>
 <segment>
-<pinref part="U$5" gate="G$1" pin="_D2"/>
-<wire x1="66.04" y1="30.48" x2="71.12" y2="30.48" width="0.1524" layer="91"/>
+<pinref part="U$5" gate="G$1" pin="_D3"/>
+<wire x1="66.04" y1="33.02" x2="71.12" y2="33.02" width="0.1524" layer="91"/>
 </segment>
 </net>
@@
 </segment>
 <segment>
-<pinref part="U$5" gate="G$1" pin="_D1"/>
-<wire x1="66.04" y1="27.94" x2="71.12" y2="27.94" width="0.1524" layer="91"/>
+<pinref part="U$5" gate="G$1" pin="_D0"/>
+<wire x1="66.04" y1="25.4" x2="71.12" y2="25.4" width="0.1524" layer="91"/>
 </segment>
 </net>
@@
 </segment>
 <segment>
-<pinref part="U$5" gate="G$1" pin="_D0"/>
-<wire x1="66.04" y1="25.4" x2="71.12" y2="25.4" width="0.1524" layer="91"/>
+<pinref part="U$5" gate="G$1" pin="_D1"/>
+<wire x1="66.04" y1="27.94" x2="71.12" y2="27.94" width="0.1524" layer="91"/>
 </segment>
 </net>
